Commit message: Fix arm mesh rendering: add GAZEBO_MODEL_PATH, remove mesh collisions that altered physics baseline, relax launch timeouts

File: src/arm_grasp_sim/urdf/arm_grasp.urdf.xacro (robot description, xacro)
@@ -76,8 +76,4 @@
       <material name="cover_plastic"/>
     </visual>
-    <collision name="base_collision">
-      <origin xyz="-0.0058789 -0.0001128 0.0294307" rpy="0 0 0"/>
-      <geometry><mesh filename="package://robomaster_description/meshes/base_collision.dae" scale="1.0 1.0 1.0"/></geometry>
-    </collision>
   </link>
   <joint name="chassis_base_joint" type="fixed">
@@ -110,8 +106,4 @@
       <material name="metal"/>
     </visual>
-    <collision name="arm_base_collision">
-      <origin xyz="-0.002098 -0.0004909 0.0073523" rpy="0 0 0"/>
-      <geometry><mesh filename="package://robomaster_description/meshes/arm_base_collision.dae" scale="1.0 1.0 1.0"/></geometry>
-    </collision>
   </link>
   <!-- ================= 肩关节 arm_1（官方原点与限位） ================= -->
@@ -139,8 +131,4 @@
       <material name="metal"/>
     </visual>
-    <collision name="arm_1_collision">
-      <origin xyz="0.0065116 0.0213649 0.0639448" rpy="0 0 0"/>
-      <geometry><mesh filename="package://robomaster_description/meshes/arm_1_collision.dae" scale="1.0 1.0 1.0"/></geometry>
-    </collision>
   </link>
   <!-- ================= 肘关节 arm_2（官方原点，限位由 rod_3 折算） ================= -->
@@ -173,8 +161,4 @@
       <material name="metal"/>
     </visual>
-    <collision name="arm_2_collision">
-      <origin xyz="0.0222614 -0.0202749 -0.008504" rpy="0 0 0"/>
-      <geometry><mesh filename="package://robomaster_description/meshes/arm_2_collision.dae" scale="1.0 1.0 1.0"/></geometry>
-    </collision>
   </link>
   <!-- ================= 末端括架（软件补偿保持水平） ================= -->
@@ -196,8 +180,4 @@
       <material name="metal"/>
     </visual>
-    <collision name="endpoint_bracket_collision">
-      <origin xyz="0.0116468 -0.0288044 0.0041342" rpy="0 0 0"/>
-      <geometry><mesh filename="package://robomaster_description/meshes/endpoint_bracket_collision.dae" scale="1.0 1.0 1.0"/></geometry>
-    </collision>
   </link>
   <!-- ================= 机械爪基座（官方） ================= -->
@@ -216,8 +196,4 @@
       <material name="EP_up.001"/>
     </visual>
-    <collision name="gripper_base_collision">
-      <origin xyz="0.0003688 -9.78e-05 -0.0112797" rpy="0 0 0"/>
-      <geometry><mesh filename="package://robomaster_description/meshes/gripper_base_collision.dae" scale="1.0 1.0 1.0"/></geometry>
-    </collision>
   </link>
   <!-- TCP（官方 gripper_t_link，用于 IK 与状态上报） -->

Commit message: 底盘加 4 个麦轮(纯视觉载体: 固定关节/无碰撞/质量1e-6, 物理基线不变, 验收 5/5)

File: src/arm_grasp_sim/urdf/arm_grasp.urdf.xacro (robot description, xacro)
@@ -28,4 +28,5 @@
   <material name="metal"><color rgba="0.0281746 0.028 0.0281746 1.0"/></material>
   <material name="EP_up.001"><color rgba="0.0284811 0.0284811 0.0284811 1.0"/></material>
+  <material name="wheel_plastic"><color rgba="0.2739087 0.2739087 0.2739087 1.0"/></material>
   <!-- ================= 世界与桌面 ================= -->
   <link name="world"/>
@@ -81,4 +82,69 @@
     <parent link="base_link"/><child link="chassis_base_link"/>
   </joint>
+  <!-- ================= 麦轮（纯视觉载体，固定关节、无碰撞、质量可忽略，不影响已验证物理） ================= -->
+    <link name="front_left_wheel_link">
+      <inertial>
+        <origin xyz="0 0 0" rpy="0 0 0"/>
+        <mass value="1e-06"/>
+        <inertia ixx="1e-09" ixy="0" ixz="0" iyy="1e-09" iyz="0" izz="1e-09"/>
+      </inertial>
+      <visual name="front_left_wheel">
+        <origin xyz="0 0 0" rpy="0 0 0"/>
+        <geometry><mesh filename="package://robomaster_description/meshes/wheel.dae" scale="1.0 1.0 1.0"/></geometry>
+        <material name="wheel_plastic"/>
+      </visual>
+    </link>
+    <joint name="front_left_wheel_joint" type="fixed">
+      <origin xyz="0.1 0.1 0.01535" rpy="0 0 0"/>
+      <parent link="chassis_base_link"/><child link="front_left_wheel_link"/>
+    </joint>
+    <link name="front_right_wheel_link">
+      <inertial>
+        <origin xyz="0 0 0" rpy="0 0 0"/>
+        <mass value="1e-06"/>
+        <inertia ixx="1e-09" ixy="0" ixz="0" iyy="1e-09" iyz="0" izz="1e-09"/>
+      </inertial>
+      <visual name="front_right_wheel">
+        <origin xyz="0 0 0" rpy="0 0 0"/>
+        <geometry><mesh filename="package://robomaster_description/meshes/wheel.dae" scale="1.0 -1.0 1.0"/></geometry>
+        <material name="wheel_plastic"/>
+      </visual>
+    </link>
+    <joint name="front_right_wheel_joint" type="fixed">
+      <origin xyz="0.1 -0.1 0.01535" rpy="0 0 0"/>
+      <parent link="chassis_base_link"/><child link="front_right_wheel_link"/>
+    </joint>
+    <link name="rear_left_wheel_link">
+      <inertial>
+        <origin xyz="0 0 0" rpy="0 0 0"/>
+        <mass value="1e-06"/>
+        <inertia ixx="1e-09" ixy="0" ixz="0" iyy="1e-09" iyz="0" izz="1e-09"/>
+      </inertial>
+      <visual name="rear_left_wheel">
+        <origin xyz="0 0 0" rpy="0 0 0"/>
+        <geometry><mesh filename="package://robomaster_description/meshes/wheel.dae" scale="1.0 -1.0 1.0"/></geometry>
+        <material name="wheel_plastic"/>
+      </visual>
+    </link>
+    <joint name="rear_left_wheel_joint" type="fixed">
+      <origin xyz="-0.1 0.1 0.01535" rpy="0 0 0"/>
+      <parent link="chassis_base_link"/><child link="rear_left_wheel_link"/>
+    </joint>
+    <link name="rear_right_wheel_link">
+      <inertial>
+        <origin xyz="0 0 0" rpy="0 0 0"/>
+        <mass value="1e-06"/>
+        <inertia ixx="1e-09" ixy="0" ixz="0" iyy="1e-09" iyz="0" izz="1e-09"/>
+      </inertial>
+      <visual name="rear_right_wheel">
+        <origin xyz="0 0 0" rpy="0 0 0"/>
+        <geometry><mesh filename="package://robomaster_description/meshes/wheel.dae" scale="1.0 1.0 1.0"/></geometry>
+        <material name="wheel_plastic"/>
+      </visual>
+    </link>
+    <joint name="rear_right_wheel_joint" type="fixed">
+      <origin xyz="-0.1 -0.1 0.01535" rpy="0 0 0"/>
+      <parent link="chassis_base_link"/><child link="rear_right_wheel_link"/>
+    </joint>
   <!-- ================= 臂基座（官方原点） ================= -->
   <joint name="arm_base_joint" type="fixed">

Commit message: 实验三: 网球/矿泉水瓶改造 — 修复网球搬运掉落(自旋螺旋爬出)
根因(实测四元数定位):
- 网球碰撞体 box 0.066 大于指盒 45x40mm, 接触合力偏离球质心,
  产生绕夹紧轴(y)的力矩 -> 球自旋(qy 0 -> -0.707)后沿指面螺旋爬出。
- 修复: 碰撞体改回 sphere r=0.033(球面法线恒过球心, 力矩恒为 0);
  指盒沿夹爪轴前移 10mm 对齐质心; 指盒加高 0.04->0.07(只向上延伸)形成笼式约束;
  kp 1e6->1e5 / kd 1->10 (0.057kg 轻体配 1e6 接触频率 667Hz 欠采样会数值爆炸);
  夹持力 25N->18N; 搬运段限速 0.45rad/s。
- 搬运位形 (0.45,-0.80)->(0.23,-0.10): 与 LIFT 位形的关节空间距离 0.893->0.347rad。
- HOME (1.30,0.35)->(0.11,0.35): 旧 HOME 指盒底 0.0611 低于瓶顶 0.125,
  转 yaw 时空夹爪把 cell_2/cell_3 的瓶推走 1.45cm 导致后续套空(即存档里"夹空"的真因)。
- 料盒内净 0.13x0.08->0.21x0.08 并补齐朝桌心一侧第 4 面墙(球体投放后会从开口滚出);
  料盒外移 r 0.21->0.24(补齐的墙会挡住 45/135 度格下降时张开的指盒, 实测格 2/3/5/6 motion_failed)。
- 同盒 3 件沿 x 错开 0.068; 投放半径钳制 0.306 + DESCEND_BIN 时长 14s(错开点半径 0.315 已到可达上限 88%)。

诚实性更正:
- gazebo_grasp_fix 插件确已构建并加载(工程内 install/, launch 已设 GAZEBO_PLUGIN_PATH),
  但实测未对本场景物体生效(物体可相对 TCP 自由移动), 不应把"不脱落"归因于它; README 已更正。
- 旧记录"球面点接触会弹飞 z=-12603"实为 kp=1e6 数值发散, 非球几何问题。

状态: 抓取链路全通, motion_failed 归零; 全任务 4/6~5/6(三次 3/6,5/6,4/6),
剩余为投放落点散布(每轮约 1 件偏 0.10~0.12m)。异常场景回归与 README 数据待更新。

File: src/arm_grasp_sim/urdf/arm_grasp.urdf.xacro (robot description, xacro)
@@ -275,5 +275,6 @@
     <parent link="gripper_link"/>
     <child link="left_finger_link"/>
-    <origin xyz="0.048 0 -0.0296" rpy="0 0 0"/>
+    <!-- x 由 0.048 前移到 0.058，使指盒中心落在被夹物质心上，见左指注释 -->
+    <origin xyz="0.058 0 -0.0296" rpy="0 0 0"/>
     <axis xyz="0 1 0"/>
     <limit effort="150" velocity="0.05" lower="0.0" upper="0.040"/>
@@ -281,12 +282,26 @@
   </joint>
   <link name="left_finger_link">
+    <!-- 指面（指盒）沿夹爪 x 轴前移 10mm：关节原点 x 由 0.048 改为 0.058。
+         根因：网球 φ0.066 被夹时指盒 x 跨度 0.045 只覆盖球的后半段，
+         指盒中心比球质心靠内 10mm，竖向支承摩擦力作用在质心后方 10mm 处，
+         对质心产生绕 y 轴（夹爪夹紧轴）的力矩，球像拨轮一样自旋
+         （实测四元数 qy 从 0 转到 -0.707，即绕 y 轴 -90°），自旋后沿指面
+         螺旋上爬直至挤出指间。前移后指盒中心正好落在被夹物质心上，力臂归零。
+         指盒中心到 TCP 的距离变为 0.066，正好等于 TCP_LEAD，与既有约定一致。
+         指盒同时在 z 向加高：由 0.04 加高到 0.07，只向上延伸（底边仍为
+         TCP-0.0106，桌面与料盒壁净空不变）。原因是搬运途中球会相对指面缓慢
+         上滑，实测球心升到 TCP+0.0397，已越过原指面顶边 TCP+0.0294，球改成骑在
+         指面顶棱上（棱接触不稳），随即持续自旋并甩出。加高后指面顶边为
+         TCP+0.0594，球心要上滑 5cm 才会骑到顶棱，笼住球。
+         注意本文件注释只能用全角标点：robot_description 是作为 ros2 的 param
+         覆盖规则交给插件解析的，半角逗号冒号双引号会让 rcl 参数解析失败。 -->
     <visual>
-      <origin xyz="0 -0.05 0" rpy="0 0 0"/>
-      <geometry><box size="0.045 0.012 0.04"/></geometry>
+      <origin xyz="0 -0.05 0.015" rpy="0 0 0"/>
+      <geometry><box size="0.045 0.012 0.07"/></geometry>
       <material name="EP_up.001"/>
     </visual>
     <collision>
-      <origin xyz="0 -0.05 0" rpy="0 0 0"/>
-      <geometry><box size="0.045 0.012 0.04"/></geometry>
+      <origin xyz="0 -0.05 0.015" rpy="0 0 0"/>
+      <geometry><box size="0.045 0.012 0.07"/></geometry>
     </collision>
     <inertial>
@@ -298,5 +313,6 @@
     <parent link="gripper_link"/>
     <child link="right_finger_link"/>
-    <origin xyz="0.048 0 -0.0296" rpy="0 0 0"/>
+    <!-- 与左指同步前移到 0.058 -->
+    <origin xyz="0.058 0 -0.0296" rpy="0 0 0"/>
     <axis xyz="0 -1 0"/>
     <limit effort="150" velocity="0.05" lower="0.0" upper="0.040"/>
@@ -304,12 +320,13 @@
   </joint>
   <link name="right_finger_link">
+    <!-- 与左指对称，指盒随关节原点前移 10mm 并加高到 0.07，见左指注释。 -->
     <visual>
-      <origin xyz="0 0.05 0" rpy="0 0 0"/>
-      <geometry><box size="0.045 0.012 0.04"/></geometry>
+      <origin xyz="0 0.05 0.015" rpy="0 0 0"/>
+      <geometry><box size="0.045 0.012 0.07"/></geometry>
       <material name="EP_up.001"/>
     </visual>
     <collision>
-      <origin xyz="0 0.05 0" rpy="0 0 0"/>
-      <geometry><box size="0.045 0.012 0.04"/></geometry>
+      <origin xyz="0 0.05 0.015" rpy="0 0 0"/>
+      <geometry><box size="0.045 0.012 0.07"/></geometry>
     </collision>
     <inertial>

Commit message: 实验三: 网球/矿泉水瓶分拣跑通 6/6 + 提交材料整理
抓取与运动
- 指节 lower 0.008 -> -0.006: 最大开口 72 -> 100mm。旧值下开口小于网球 φ66,
  每侧只剩 3mm, 叠加实测 10.8mm 指心定位误差 -> 下降必撞开物体 -> 合爪零接触(夹空)。
  改后 grasp_failed 由 5 例降为 0, 此后所有轮次稳定为 0。
- 6 格整体外移 r=0.185 -> 0.225 (launch/server/grid_mapper/world 四处坐标同步)。
- 料盒改 0.29x0.29 正方; 近壁与两侧壁顶削到 z=0.040: 张开 100mm 的指盒在对角格
  扫掠最远 |y|=0.2188 已越过近墙 y=0.1925 (正前/正后格只到 0.062, 故历史上只有
  cell_1/cell_4 能成)。按高度避让而非 xy 余量(当时余量仅 0.3mm)。
- Z_DROP 0.115 -> 0.095: 壁顶削矮后不需要高抛, 原值等于 8.7cm 自由落体会把瓶
  弹出矮壁盒(实测 dist=0.084 判 place_failed)。
- 瓶身 phi65 -> phi55, collision 外接盒同步 0.055 0.055 0.10 (只改 visual 会留下
  隐形的大碰撞盒)。

失败隔离
- RELEASE 开爪窗口 2s -> 3s; 每格 HOME 后新增 _ensure_palm_clear(): 扫描 6 个物体,
  任一 z>0.105 判为上一格漏脱焊, 强制开爪 3s 最多 3 次。
- SCAN 稳定窗口改为"出现本轮未见过的网格即重开"(scan_reopen_cap=20s): 原逻辑从进入
  SCAN 起算、只在桌面全空时重置, 首批检测一到就定计划, 6 路并行 spawn 中最晚的两个
  物体被整轮记成"空网格"(实测 4/6)。顺带补 scan_enter_t 初值(原只在 _kick 赋值,
  第 1 秒内来检测会 AttributeError)。

材料
- docs/实验三_提交材料/: 提交清单索引、检测与网格配置说明、状态机配置 XML、
  9/22 验收日志与各轮汇总、4 个异常场景记录、简要实验报告、视频说明。
- patches/robomaster_ros_local_fixes.patch + scripts/fix_rm_mesh_texture.sh:
  submodule 本地改动与网格贴图引用名错误(EP_all_01_b_png 少个点)无法随父仓库上传,
  改为导出补丁 + 幂等修复脚本, README 补"克隆后必要前置步骤"。
- 首次纳入 run_exceptions.sh / classify_real.* / gazebo_mimic_plugin 等此前未跟踪的交付物。
- models/best_real3.onnx 按直接提交方式交付(38MB)。
- .gitignore 增加 *.bak* / *_bak / *.orig / *.rej / *.pt 等。

结论订正
- README 原写"实测 gazebo_grasp_fix 对本场景不生效、不要把不掉落归因于它", 该结论
  已被对照实跑否证: 插件确实生效(日志 attach/detach 与抓取一一对应); 关掉它仍 5/6
  placed, 说明摩擦夹持本身成立但纯摩擦做不到 6/6。
- 真机: 实验二定点抓取有实机记录(videos/real_grasp_5of5.mp4 + logs/real_machine 5 份
  SUCCESS CSV), 实验三分类流程未上真机。

验收
placed=6 failed=0 skipped=0; unreachable/grasp_failed/motion_failed/place_failed 均 0;
带 gzclient 整轮 318s, RTF 约 1.25; attach/detach 6/6 配平。

File: src/arm_grasp_sim/urdf/arm_grasp.urdf.xacro (robot description, xacro)
@@ -178,5 +178,5 @@
     <parent link="arm_base_link"/><child link="arm_1_link"/>
     <axis xyz="0.0 1.0 0"/>
-    <limit effort="6" velocity="3" lower="-0.274" upper="1.384"/>
+    <limit effort="12" velocity="3" lower="-0.274" upper="1.384"/>
     <dynamics damping="1.0"/>
   </joint>
@@ -203,5 +203,5 @@
     <parent link="arm_1_link"/><child link="arm_2_link"/>
     <axis xyz="0.0 1.0 0"/>
-    <limit effort="6" velocity="3" lower="-1.25" upper="0.40"/>
+    <limit effort="12" velocity="3" lower="-1.25" upper="0.40"/>
     <dynamics damping="1.0"/>
   </joint>
@@ -278,5 +278,5 @@
     <origin xyz="0.058 0 -0.0296" rpy="0 0 0"/>
     <axis xyz="0 1 0"/>
-    <limit effort="150" velocity="0.05" lower="0.0" upper="0.040"/>
+    <limit effort="150" velocity="0.05" lower="-0.006" upper="0.040"/>
     <dynamics damping="0.5" friction="0.2"/>
   </joint>
@@ -316,5 +316,5 @@
     <origin xyz="0.058 0 -0.0296" rpy="0 0 0"/>
     <axis xyz="0 -1 0"/>
-    <limit effort="150" velocity="0.05" lower="0.0" upper="0.040"/>
+    <limit effort="150" velocity="0.05" lower="-0.006" upper="0.040"/>
     <dynamics damping="0.5" friction="0.2"/>
   </joint>

File: src/arm_grasp_sim/urdf/bottle.urdf (robot description, URDF)
Before this commit: robot bottle, 1 links, 0 joints
Links:
- link bottle: geometry collision box size=0.055 0.055 0.10; visual cylinder length=0.02 radius=0.015
